File: crossover.kicad_pcb (KiCad board)
At the start: 2 copper layers, 78 parts, among them J1 Power In, J2 Line In, J3 Tweeter Out, J4 Sub Out, U1 TL072, U2 TL072, U3 TL072, U4 TL072, U5 TL072, U6 TL072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

Commit message: Set boundaries, labels
Parts:
- added TP1: L HPF, TestPoint:TestPoint_Pad_1.0x1.0mm, F.Cu at (126.5, 35.3)
- added TP2: L LPF, TestPoint:TestPoint_Pad_1.0x1.0mm, F.Cu at (102.2, 82.6)
- added TP3: R HPF, TestPoint:TestPoint_Pad_1.0x1.0mm, F.Cu at (114.0, 56.6)
- added TP4: R LPF, TestPoint:TestPoint_Pad_1.0x1.0mm, F.Cu at (127.4, 91.1)
- moved R6 23.1 mm to (97.3, 70.8), turned to -90 degrees
- moved C32 13.6 mm to (151.8, 72.8)
- moved R5 10.5 mm to (97.3, 67.9), turned to 90 degrees
- moved U1 7.18 mm to (84.9, 60.8)
- moved R4 7.15 mm to (79.9, 60.9), turned to -90 degrees
- moved C16 6.66 mm to (92.7, 72.9)
- moved C29 3.71 mm to (71.8, 56.6)
- moved J2 3.68 mm to (65.8, 61.4)
- moved C28 2.82 mm to (72.0, 64.6)
- moved J4 2.24 mm to (158.5, 69.5), turned to -90 degrees
- moved C26 2.13 mm to (147.2, 69.1)
- moved R13 1.79 mm to (123.3, 56.2)
- moved R25 1.51 mm to (91.4, 52.8)
- moved R26 1.51 mm to (91.3, 42.8)
- moved R3 1.26 mm to (86.7, 55.9)
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Other:
- board outline added: 99.7 x 90.8 mm
- board text added: "+"
- board text added: "-"
- board text added: "L"
- board text added: "Left"
- board text added: "R"
- board text added: "Right"
- board text added: "Sub"

Commit message: Fully routed
Parts:
- added REF**: MountingHole_3.2mm_M3, MountingHole:MountingHole_3.2mm_M3, F.Cu at (158.8, 30.3)
- added REF**: MountingHole_3.2mm_M3, MountingHole:MountingHole_3.2mm_M3, F.Cu at (66.3, 113.2)
- added REF**: MountingHole_3.2mm_M3, MountingHole:MountingHole_3.2mm_M3, F.Cu at (66.6, 30.1)
- added REF**: MountingHole_3.2mm_M3, MountingHole:MountingHole_3.2mm_M3, F.Cu at (158.6, 113.3)
- moved C3 24.9 mm to (124.0, 31.0), turned to 180 degrees
- moved C4 0.23 mm to (115.2, 31.1)
Routing:
- net VCC: track 0.00 -> 298.6 mm, vias 0 -> 3
- net VDD: track 0.00 -> 287.3 mm, vias 0 -> 2
- net /Left Gain/in: track 0.00 -> 76.5 mm
- net /Left LPF/out: track 0.00 -> 70.1 mm
- net GNDREF: track 0.00 -> 53.6 mm, vias 0 -> 2
- net /Right HPF/out: track 0.00 -> 49.1 mm, vias 0 -> 2
- net /Left HPF/HPF Stage 2/in: track 0.00 -> 37.6 mm, vias 0 -> 1
- net /Left HPF/in: track 0.00 -> 35.1 mm, vias 0 -> 1
- net /Right HPF/in: track 0.00 -> 32.9 mm
- net /Right gain/out: track 0.00 -> 25.5 mm
- net /Right Input Buffer/In: track 0.00 -> 25.4 mm
- net Net-(R27-Pad1): track 0.00 -> 24.3 mm
- net /sub gain/in: track 0.00 -> 23.6 mm
- net /Right LPF/out: track 0.00 -> 23.0 mm
- net Net-(R29-Pad1): track 0.00 -> 22.7 mm
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- added copper zone on B.Cu, net GNDREF
- added copper zone on B.Cu, net VDD

Commit message: Final PCB Layout
Routing:
- net VDD: vias 2 -> 1
- net GNDREF: vias 2 -> 0
Other:
- board text added: "Audio Crossover v1.0 Circuit: https://sound-au.com/project09.htm"
Changed lines of the file:
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@@
       (layerselection 0x00010fc_ffffffff)
       (disableapertmacros false)
-      (usegerberextensions false)
+      (usegerberextensions true)
       (usegerberattributes true)
       (usegerberadvancedattributes true)
@@
       (psa4output false)
       (plotreference true)
-      (plotvalue true)
+      (plotvalue false)
       (plotinvisibletext false)
       (sketchpadsonfab false)
@@
       (outputformat 1)
       (mirror false)
-      (drillshape 1)
+      (drillshape 0)
       (scaleselection 1)
-      (outputdirectory "")
+      (outputdirectory "build/")
     )
   )
@@
     (fp_line (start -2.91 2.61) (end -0.41 2.61) (layer "F.Fab") (width 0.1))
     (fp_line (start 7.5 -1.6) (end -2.5 -1.6) (layer "F.Fab") (width 0.1))
-    (pad "1" thru_hole roundrect (at 0 0 180) (size 1.7 1.95) (drill 0.95) (layers *.Cu *.Mask) (roundrect_rratio 0.147059)
+    (pad "1" thru_hole roundrect (at 0 0 180) (size 1.7 1.95) (drill 0.95) (layers *.Cu *.Mask) (roundrect_rratio 0.1470588235)
       (net 33 "Net-(C30-Pad2)") (pinfunction "Pin_1") (pintype "passive"))
     (pad "2" thru_hole oval (at 2.5 0 180) (size 1.7 1.95) (drill 0.95) (layers *.Cu *.Mask)
@@
     (fp_line (start 7.5 -1.6) (end -2.5 -1.6) (layer "F.Fab") (width 0.1))
     (fp_line (start -2.5 -1.6) (end -2.5 2.2) (layer "F.Fab") (width 0.1))
-    (pad "1" thru_hole roundrect (at 0 0 90) (size 1.7 1.95) (drill 0.95) (layers *.Cu *.Mask) (roundrect_rratio 0.147059)
+    (pad "1" thru_hole roundrect (at 0 0 90) (size 1.7 1.95) (drill 0.95) (layers *.Cu *.Mask) (roundrect_rratio 0.1470588235)
       (net 28 "Net-(C28-Pad1)") (pinfunction "Pin_1") (pintype "passive"))
     (pad "2" thru_hole oval (at 2.5 0 90) (size 1.7 1.95) (drill 0.95) (layers *.Cu *.Mask)
@@
     (fp_line (start -2.91 2.61) (end -0.41 2.61) (layer "F.Fab") (width 0.1))
     (fp_line (start -2.91 0.11) (end -2.91 2.61) (layer "F.Fab") (width 0.1))
-    (pad "1" thru_hole roundrect (at 0 0 270) (size 1.7 2) (drill 1) (layers *.Cu *.Mask) (roundrect_rratio 0.147059)
+    (pad "1" thru_hole roundrect (at 0 0 270) (size 1.7 2) (drill 1) (layers *.Cu *.Mask) (roundrect_rratio 0.1470588235)
       (net 37 "Net-(C32-Pad2)") (pinfunction "Pin_1") (pintype "passive"))
     (pad "2" thru_hole oval (at 2.5 0 270) (size 1.7 2) (drill 1) (layers *.Cu *.Mask)
@@
     (fp_line (start -2.5 -1.6) (end -2.5 2.2) (layer "F.Fab") (width 0.1))
     (fp_line (start 5 2.2) (end 5 -1.6) (layer "F.Fab") (width 0.1))
-    (pad "1" thru_hole roundrect (at 0 0 90) (size 1.7 2) (drill 1) (layers *.Cu *.Mask) (roundrect_rratio 0.147059)
+    (pad "1" thru_hole roundrect (at 0 0 90) (size 1.7 2) (drill 1) (layers *.Cu *.Mask) (roundrect_rratio 0.1470588235)
       (net 21 "VCC") (pinfunction "Pin_1") (pintype "passive"))
     (pad "2" thru_hole oval (at 2.5 0 90) (size 1.7 2) (drill 1) (layers *.Cu *.Mask)
@@
   )
   (gr_rect (start 62.815202 26.482667) (end 162.480869 117.232856) (layer "Edge.Cuts") (width 0.1) (fill none))
+  (gr_text "Audio Crossover v1.0\nCircuit: https://sound-au.com/project09.htm\n" (at 95.87642 109.351939) (layer "B.SilkS")
+    (effects (font (size 0.635 0.635) (thickness 0.15875)) (justify left mirror))
+  )
   (gr_text "R" (at 65.75669 65.670123 270) (layer "F.SilkS")
     (effects (font (size 1.5 1.5) (thickness 0.3)))
@@
   (segment (start 97.650507 35.182083) (end 99.505042 37.036618) (width 0.25) (layer "F.Cu") (net 22))
   (segment (start 125.146776 45.18527) (end 138.655893 31.676153) (width 0.25) (layer "F.Cu") (net 22))
-  (via (at 64.906846 51.344079) (size 0.8) (drill 0.4) (layers "F.Cu" "B.Cu") (net 22))
   (via (at 148.276825 77.175671) (size 0.8) (drill 0.4) (layers "F.Cu" "B.Cu") (net 22))
   (segment (start 125.146776 46.960016) (end 121.697476 46.960016) (width 0.25) (layer "B.Cu") (net 22))
@@
   (segment (start 128.214322 65.985595) (end 137.334979 65.985595) (width 0.25) (layer "B.Cu") (net 22))
   (segment (start 121.58753 74.800606) (end 127.25584 69.132296) (width 0.25) (layer "B.Cu") (net 22))
-  (via (at 127.847332 63.588598) (size 0.8) (drill 0.4) (layers "F.Cu" "B.Cu") (net 23))
-  (via (at 97.277488 43.928461) (size 0.8) (drill 0.4) (layers "F.Cu" "B.Cu") (free) (net 23))
   (segment (start 83.401138 46.399929) (end 83.334831 46.466236) (width 0.25) (layer "B.Cu") (net 23))
   (segment (start 89.006015 43.792495) (end 90.041548 43.792495) (width 0.25) (layer "B.Cu") (net 23))
