File: crossover.kicad_sch (KiCad schematic)
At the start: 12 parts, among them J1 Power In, J2 Line In, J3 Tweeter Out, J4 Sub Out, U6 TL072

Commit message: Set boundaries, labels
Parts:
- added TP1: L HPF, TestPoint:TestPoint_Pad_1.0x1.0mm, symbol Connector:TestPoint
- added TP2: L LPF, TestPoint:TestPoint_Pad_1.0x1.0mm, symbol Connector:TestPoint
- added TP3: R HPF, TestPoint:TestPoint_Pad_1.0x1.0mm, symbol Connector:TestPoint
- added TP4: R LPF, TestPoint:TestPoint_Pad_1.0x1.0mm, symbol Connector:TestPoint
- U6: footprint (none) -> Package_DIP:DIP-8_W7.62mm_Socket
Connections:
- net Left Gain/in: now also TP1.1
- net Left LPF/out: now also TP2.1
- net Right HPF/out: now also TP3.1
- net Right LPF/out: now also TP4.1
Changed lines of the file:
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@@
 (kicad_sch (version 20211123) (generator eeschema)
   (paper "A4")
+  (junction (at 200.66 57.15) (diameter 0) (color 0 0 0 0)
+  )
+  (junction (at 208.28 153.67) (diameter 0) (color 0 0 0 0)
+  )
   (junction (at 146.05 121.92) (diameter 0) (color 0 0 0 0)
   )
+  (junction (at 201.93 120.65) (diameter 0) (color 0 0 0 0)
+  )
   (junction (at 137.16 63.5) (diameter 0) (color 0 0 0 0)
+  )
+  (junction (at 201.93 92.71) (diameter 0) (color 0 0 0 0)
   )
   (junction (at 220.98 113.03) (diameter 0) (color 0 0 0 0)
@@
   (no_connect (at 105.41 171.45))
   (no_connect (at 90.17 173.99))
+  (wire (pts (xy 201.93 92.71) (xy 220.98 92.71))
+    (stroke (width 0) (type default) (color 0 0 0 0))
+  )
   (wire (pts (xy 271.78 50.8) (xy 271.78 53.34))
     (stroke (width 0) (type default) (color 0 0 0 0))
@@
     (stroke (width 0) (type default) (color 0 0 0 0))
   )
-  (wire (pts (xy 195.58 120.65) (xy 210.82 120.65))
+  (wire (pts (xy 195.58 120.65) (xy 201.93 120.65))
     (stroke (width 0) (type default) (color 0 0 0 0))
   )
@@
     (stroke (width 0) (type default) (color 0 0 0 0))
   )
-  (wire (pts (xy 195.58 92.71) (xy 220.98 92.71))
+  (wire (pts (xy 195.58 92.71) (xy 201.93 92.71))
     (stroke (width 0) (type default) (color 0 0 0 0))
   )
@@
     (stroke (width 0) (type default) (color 0 0 0 0))
   )
-  (wire (pts (xy 199.39 57.15) (xy 207.01 57.15))
+  (wire (pts (xy 199.39 57.15) (xy 200.66 57.15))
     (stroke (width 0) (type default) (color 0 0 0 0))
   )
@@
     (stroke (width 0) (type default) (color 0 0 0 0))
   )
+  (wire (pts (xy 200.66 57.15) (xy 207.01 57.15))
+    (stroke (width 0) (type default) (color 0 0 0 0))
+  )
   (wire (pts (xy 146.05 120.65) (xy 154.94 120.65))
     (stroke (width 0) (type default) (color 0 0 0 0))
   )
+  (wire (pts (xy 208.28 153.67) (xy 220.98 153.67))
+    (stroke (width 0) (type default) (color 0 0 0 0))
+  )
   (wire (pts (xy 154.94 93.98) (xy 137.16 93.98))
     (stroke (width 0) (type default) (color 0 0 0 0))
@@
     (stroke (width 0) (type default) (color 0 0 0 0))
   )
-  (wire (pts (xy 199.39 153.67) (xy 220.98 153.67))
+  (wire (pts (xy 199.39 153.67) (xy 208.28 153.67))
+    (stroke (width 0) (type default) (color 0 0 0 0))
+  )
+  (wire (pts (xy 201.93 120.65) (xy 210.82 120.65))
     (stroke (width 0) (type default) (color 0 0 0 0))
   )
@@
     (pin "3")
   )
+  (symbol (lib_id "Connector:TestPoint") (at 201.93 92.71 0) (unit 1)
+    (in_bom yes) (on_board yes) (fields_autoplaced)
+    (property "Reference" "TP2" (id 0) (at 204.47 88.1379 0)
+      (effects (font (size 1.27 1.27)) (justify left))
+    )
+    (property "Value" "L LPF" (id 1) (at 204.47 90.6779 0)
+      (effects (font (size 1.27 1.27)) (justify left))
+    )
+    (property "Footprint" "TestPoint:TestPoint_Pad_1.0x1.0mm" (id 2) (at 207.01 92.71 0)
+      (effects (font (size 1.27 1.27)) hide)
+    )
+    (property "Datasheet" "~" (id 3) (at 207.01 92.71 0)
+      (effects (font (size 1.27 1.27)) hide)
+    )
+    (pin "1")
+  )
   (symbol (lib_id "Amplifier_Operational:TL072") (at 97.79 171.45 0) (unit 2)
     (in_bom yes) (on_board yes) (fields_autoplaced)
     (property "Reference" "U6" (id 0) (at 97.79 161.29 0))
     (property "Value" "TL072" (id 1) (at 97.79 163.83 0))
-    (property "Footprint" "" (id 2) (at 97.79 171.45 0)
+    (property "Footprint" "Package_DIP:DIP-8_W7.62mm_Socket" (id 2) (at 97.79 171.45 0)
       (effects (font (size 1.27 1.27)) hide)
     )
@@
     (pin "1")
   )
+  (symbol (lib_id "Connector:TestPoint") (at 201.93 120.65 0) (unit 1)
+    (in_bom yes) (on_board yes) (fields_autoplaced)
+    (property "Reference" "TP3" (id 0) (at 204.47 116.0779 0)
+      (effects (font (size 1.27 1.27)) (justify left))
+    )
+    (property "Value" "R HPF" (id 1) (at 204.47 118.6179 0)
+      (effects (font (size 1.27 1.27)) (justify left))
+    )
+    (property "Footprint" "TestPoint:TestPoint_Pad_1.0x1.0mm" (id 2) (at 207.01 120.65 0)
+      (effects (font (size 1.27 1.27)) hide)
+    )
+    (property "Datasheet" "~" (id 3) (at 207.01 120.65 0)
+      (effects (font (size 1.27 1.27)) hide)
+    )
+    (pin "1")
+  )
   (symbol (lib_id "Connector:Conn_01x02_Male") (at 20.32 33.02 0) (unit 1)
     (in_bom yes) (on_board yes) (fields_autoplaced)
@@
     (pin "2")
   )
+  (symbol (lib_id "Connector:TestPoint") (at 200.66 57.15 0) (unit 1)
+    (in_bom yes) (on_board yes)
+    (property "Reference" "TP1" (id 0) (at 199.39 55.88 0)
+      (effects (font (size 1.27 1.27)) (justify left))
+    )
+    (property "Value" "L HPF" (id 1) (at 198.12 52.07 0)
+      (effects (font (size 1.27 1.27)) (justify left))
+    )
+    (property "Footprint" "TestPoint:TestPoint_Pad_1.0x1.0mm" (id 2) (at 205.74 57.15 0)
+      (effects (font (size 1.27 1.27)) hide)
+    )
+    (property "Datasheet" "~" (id 3) (at 205.74 57.15 0)
+      (effects (font (size 1.27 1.27)) hide)
+    )
+    (pin "1")
+  )
   (symbol (lib_id "power:VDD") (at 271.78 53.34 180) (unit 1)
     (in_bom yes) (on_board yes) (fields_autoplaced)
@@
     (pin "1")
     (pin "2")
+  )
+  (symbol (lib_id "Connector:TestPoint") (at 208.28 153.67 0) (unit 1)
+    (in_bom yes) (on_board yes) (fields_autoplaced)
+    (property "Reference" "TP4" (id 0) (at 210.82 149.0979 0)
+      (effects (font (size 1.27 1.27)) (justify left))
+    )
+    (property "Value" "R LPF" (id 1) (at 210.82 151.6379 0)
+      (effects (font (size 1.27 1.27)) (justify left))
+    )
+    (property "Footprint" "TestPoint:TestPoint_Pad_1.0x1.0mm" (id 2) (at 213.36 153.67 0)
+      (effects (font (size 1.27 1.27)) hide)
+    )
+    (property "Datasheet" "~" (id 3) (at 213.36 153.67 0)
+      (effects (font (size 1.27 1.27)) hide)
+    )
+    (pin "1")
   )
   (symbol (lib_id "Device:C_Polarized_Small_US") (at 55.88 90.17 0) (unit 1)
@@
       (reference "RV3") (unit 1) (value "10K") (footprint "Potentiometer_THT:Potentiometer_Bourns_3386C_Horizontal")
     )
+    (path "/c04556e4-a163-441b-8f32-1c9ceaa7e44c"
+      (reference "TP1") (unit 1) (value "L HPF") (footprint "TestPoint:TestPoint_Pad_1.0x1.0mm")
+    )
+    (path "/06af92dc-ad44-4a47-8328-293a3179d3bb"
+      (reference "TP2") (unit 1) (value "L LPF") (footprint "TestPoint:TestPoint_Pad_1.0x1.0mm")
+    )
+    (path "/b4d97c9e-7d50-447a-8f4e-837052683056"
+      (reference "TP3") (unit 1) (value "R HPF") (footprint "TestPoint:TestPoint_Pad_1.0x1.0mm")
+    )
+    (path "/d231025d-16de-4192-aeac-047f3abf3bfa"
+      (reference "TP4") (unit 1) (value "R LPF") (footprint "TestPoint:TestPoint_Pad_1.0x1.0mm")
+    )
     (path "/87eeb169-ec39-4325-b98a-d89c839087c5/0c33cd70-ebd7-4f01-b33d-b6dee68b2571"
       (reference "U1") (unit 1) (value "TL072") (footprint "Package_DIP:DIP-8_W7.62mm_Socket")
@@
     )
     (path "/13343b0a-3170-4d29-a2cc-ffa359b95298"
-      (reference "U6") (unit 2) (value "TL072") (footprint "")
+      (reference "U6") (unit 2) (value "TL072") (footprint "Package_DIP:DIP-8_W7.62mm_Socket")
     )
     (path "/71d523ed-d1c3-4d8e-9d3a-4faa4d6820b4/b41c02f7-a817-4cc4-8c21-969ab3ae800b"
