File: crossover.kicad_sch (KiCad schematic)
At the start: 9 parts, among them J1 Power In, J2 Line In, J3 Tweeter Out, J4 Sub Out

Commit message: Finished routing
Connections:
- net Left Gain/out: now also J3.3 (Pin_3); no longer J3.1 (Pin_1)
- net Right gain/out: now also J3.1 (Pin_1); no longer J3.3 (Pin_3)
Changed lines of the file:
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@@
-    (stroke (width 0) (type default))
-  )
-  (wire (pts (xy 254 78.74) (xy 254 53.34))
     (stroke (width 0) (type default))
   )
@@
     (stroke (width 0) (type default))
   )
-  (wire (pts (xy 227.33 55.88) (xy 233.68 55.88))
-    (stroke (width 0) (type default))
-  )
   (wire (pts (xy 123.19 63.5) (xy 137.16 63.5))
     (stroke (width 0) (type default))
   )
-  (wire (pts (xy 236.22 78.74) (xy 254 78.74))
+  (wire (pts (xy 236.22 78.74) (xy 257.81 78.74))
     (stroke (width 0) (type default))
   )
@@
     (stroke (width 0) (type default))
   )
-  (wire (pts (xy 233.68 48.26) (xy 233.68 55.88))
-    (stroke (width 0) (type default))
-  )
   (wire (pts (xy 146.05 121.92) (xy 146.05 120.65))
     (stroke (width 0) (type default))
@@
     (stroke (width 0) (type default))
   )
+  (wire (pts (xy 227.33 55.88) (xy 254 55.88))
+    (stroke (width 0) (type default))
+  )
   (wire (pts (xy 271.78 116.84) (xy 273.05 116.84))
     (stroke (width 0) (type default))
@@
     (stroke (width 0) (type default))
   )
-  (wire (pts (xy 233.68 48.26) (xy 254 48.26))
-    (stroke (width 0) (type default))
-  )
   (wire (pts (xy 55.88 109.22) (xy 93.98 124.46))
     (stroke (width 0) (type default))
@@
     (stroke (width 0) (type default))
   )
+  (wire (pts (xy 254 55.88) (xy 254 53.34))
+    (stroke (width 0) (type default))
+  )
   (wire (pts (xy 267.97 114.3) (xy 273.05 114.3))
     (stroke (width 0) (type default))
@@
     (stroke (width 0) (type default))
   )
+  (wire (pts (xy 257.81 48.26) (xy 254 48.26))
+    (stroke (width 0) (type default))
+  )
   (wire (pts (xy 227.33 132.08) (xy 227.33 142.24))
     (stroke (width 0) (type default))
@@
   )
   (wire (pts (xy 210.82 80.01) (xy 215.9 80.01))
+    (stroke (width 0) (type default))
+  )
+  (wire (pts (xy 257.81 78.74) (xy 257.81 48.26))
     (stroke (width 0) (type default))
   )
@@
   )
   (symbol (lib_id "Device:R") (at 241.3 142.24 90) (unit 1)
-    (in_bom yes) (on_board yes) (dnp no) (fields_autoplaced)
+    (in_bom yes) (on_board yes) (dnp no)
     (property "Reference" "R3" (at 241.3 137.16 90)
       (effects (font (size 1.27 1.27)))
@@
   )
   (symbol (lib_id "Device:R") (at 220.98 119.38 0) (unit 1)
-    (in_bom yes) (on_board yes) (dnp no) (fields_autoplaced)
+    (in_bom yes) (on_board yes) (dnp no)
     (property "Reference" "R2" (at 223.52 118.1099 0)
       (effects (font (size 1.27 1.27)) (justify left))
