File: gain.kicad_sch (KiCad schematic)
At the start: 5 parts, among them U7 TL072

Commit message: Final PCB Layout
Parts:
- R32: value 5k -> 10K
Changed lines of the file:
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@@
       (effects (font (size 1.27 1.27)) (justify left))
     )
-    (property "Value" "5k" (id 1) (at 92.71 83.8199 0)
+    (property "Value" "10K" (id 1) (at 92.71 83.8199 0)
       (effects (font (size 1.27 1.27)) (justify left))
     )
