File: hpf_1_stage.kicad_sch (KiCad schematic)
At the start: 5 parts, among them U2 TL072

Commit message: Final PCB Layout
Parts:
- R7: value 56K -> 39K
- R8: value 27K -> 20K
Changed lines of the file:
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@@
     (in_bom yes) (on_board yes) (fields_autoplaced)
     (property "Reference" "R8" (id 0) (at 99.06 41.91 90))
-    (property "Value" "27K" (id 1) (at 99.06 44.45 90))
+    (property "Value" "20K" (id 1) (at 99.06 44.45 90))
     (property "Footprint" "Resistor_THT:R_Axial_DIN0207_L6.3mm_D2.5mm_P7.62mm_Horizontal" (id 2) (at 99.06 50.038 90)
       (effects (font (size 1.27 1.27)) hide)
@@
       (effects (font (size 1.27 1.27)) (justify left))
     )
-    (property "Value" "56K" (id 1) (at 93.98 69.8499 0)
+    (property "Value" "39K" (id 1) (at 93.98 69.8499 0)
       (effects (font (size 1.27 1.27)) (justify left))
     )
