File: lpf 1 stage.kicad_sch (KiCad schematic)
At the start: 5 parts, among them U4 TL072

Commit message: Final PCB Layout
Parts:
- R15, R16: value 27K -> 20K
Changed lines of the file:
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@@
     (in_bom yes) (on_board yes) (fields_autoplaced)
     (property "Reference" "R15" (id 0) (at 80.01 59.69 90))
-    (property "Value" "27K" (id 1) (at 80.01 62.23 90))
+    (property "Value" "20K" (id 1) (at 80.01 62.23 90))
     (property "Footprint" "Resistor_THT:R_Axial_DIN0207_L6.3mm_D2.5mm_P7.62mm_Horizontal" (id 2) (at 80.01 67.818 90)
       (effects (font (size 1.27 1.27)) hide)
@@
     (in_bom yes) (on_board yes) (fields_autoplaced)
     (property "Reference" "R16" (id 0) (at 95.25 59.69 90))
-    (property "Value" "27K" (id 1) (at 95.25 62.23 90))
+    (property "Value" "20K" (id 1) (at 95.25 62.23 90))
     (property "Footprint" "Resistor_THT:R_Axial_DIN0207_L6.3mm_D2.5mm_P7.62mm_Horizontal" (id 2) (at 95.25 67.818 90)
       (effects (font (size 1.27 1.27)) hide)
