File: lpf 1 stage.kicad_sch (KiCad schematic)
At the start: 5 parts, among them U4 TL072

Commit message: Re-annotate and run erc
Parts:
- renumbered C22 to C13, C9 to C14, R15 to R18, R16 to R19
Changed lines of the file:
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@@
   (symbol (lib_id "power:GNDREF") (at 100.33 80.01 0) (unit 1)
     (in_bom yes) (on_board yes) (dnp no) (fields_autoplaced)
-    (property "Reference" "#PWR010" (at 100.33 86.36 0)
+    (property "Reference" "#PWR013" (at 100.33 86.36 0)
       (effects (font (size 1.27 1.27)) hide)
     )
@@
       (project "crossover"
         (path "/3c8df2a5-e9f9-4495-af40-aa221f0b3fa5/4179ae51-cf3a-4bce-929c-a59c2a13f09f/f3a16da1-c1d9-43a4-8a05-0965021b6865"
-          (reference "#PWR010") (unit 1)
-        )
-        (path "/3c8df2a5-e9f9-4495-af40-aa221f0b3fa5/4179ae51-cf3a-4bce-929c-a59c2a13f09f/162d0e00-6252-4458-837d-88970c658cfc"
-          (reference "#PWR011") (unit 1)
-        )
-        (path "/3c8df2a5-e9f9-4495-af40-aa221f0b3fa5/8cd80f45-633d-420a-bdbe-39ad6abe5b0e/f3a16da1-c1d9-43a4-8a05-0965021b6865"
-          (reference "#PWR012") (unit 1)
-        )
-        (path "/3c8df2a5-e9f9-4495-af40-aa221f0b3fa5/8cd80f45-633d-420a-bdbe-39ad6abe5b0e/162d0e00-6252-4458-837d-88970c658cfc"
           (reference "#PWR013") (unit 1)
         )
+        (path "/3c8df2a5-e9f9-4495-af40-aa221f0b3fa5/4179ae51-cf3a-4bce-929c-a59c2a13f09f/162d0e00-6252-4458-837d-88970c658cfc"
+          (reference "#PWR014") (unit 1)
+        )
+        (path "/3c8df2a5-e9f9-4495-af40-aa221f0b3fa5/8cd80f45-633d-420a-bdbe-39ad6abe5b0e/f3a16da1-c1d9-43a4-8a05-0965021b6865"
+          (reference "#PWR015") (unit 1)
+        )
+        (path "/3c8df2a5-e9f9-4495-af40-aa221f0b3fa5/8cd80f45-633d-420a-bdbe-39ad6abe5b0e/162d0e00-6252-4458-837d-88970c658cfc"
+          (reference "#PWR016") (unit 1)
+        )
       )
     )
@@
   (symbol (lib_id "Device:C") (at 104.14 53.34 90) (unit 1)
     (in_bom yes) (on_board yes) (dnp no) (fields_autoplaced)
-    (property "Reference" "C9" (at 104.14 45.72 90)
+    (property "Reference" "C14" (at 104.14 45.72 90)
       (effects (font (size 1.27 1.27)))
     )
@@
       (project "crossover"
         (path "/3c8df2a5-e9f9-4495-af40-aa221f0b3fa5/4179ae51-cf3a-4bce-929c-a59c2a13f09f/f3a16da1-c1d9-43a4-8a05-0965021b6865"
-          (reference "C9") (unit 1)
-        )
-        (path "/3c8df2a5-e9f9-4495-af40-aa221f0b3fa5/4179ae51-cf3a-4bce-929c-a59c2a13f09f/162d0e00-6252-4458-837d-88970c658cfc"
-          (reference "C10") (unit 1)
-        )
-        (path "/3c8df2a5-e9f9-4495-af40-aa221f0b3fa5/8cd80f45-633d-420a-bdbe-39ad6abe5b0e/f3a16da1-c1d9-43a4-8a05-0965021b6865"
-          (reference "C11") (unit 1)
-        )
-        (path "/3c8df2a5-e9f9-4495-af40-aa221f0b3fa5/8cd80f45-633d-420a-bdbe-39ad6abe5b0e/162d0e00-6252-4458-837d-88970c658cfc"
-          (reference "C12") (unit 1)
+          (reference "C14") (unit 1)
+        )
+        (path "/3c8df2a5-e9f9-4495-af40-aa221f0b3fa5/4179ae51-cf3a-4bce-929c-a59c2a13f09f/162d0e00-6252-4458-837d-88970c658cfc"
+          (reference "C16") (unit 1)
+        )
+        (path "/3c8df2a5-e9f9-4495-af40-aa221f0b3fa5/8cd80f45-633d-420a-bdbe-39ad6abe5b0e/f3a16da1-c1d9-43a4-8a05-0965021b6865"
+          (reference "C18") (unit 1)
+        )
+        (path "/3c8df2a5-e9f9-4495-af40-aa221f0b3fa5/8cd80f45-633d-420a-bdbe-39ad6abe5b0e/162d0e00-6252-4458-837d-88970c658cfc"
+          (reference "C20") (unit 1)
         )
       )
@@
   (symbol (lib_id "Device:R") (at 80.01 66.04 90) (unit 1)
     (in_bom yes) (on_board yes) (dnp no) (fields_autoplaced)
-    (property "Reference" "R15" (at 80.01 59.69 90)
+    (property "Reference" "R18" (at 80.01 59.69 90)
       (effects (font (size 1.27 1.27)))
     )
@@
       (project "crossover"
         (path "/3c8df2a5-e9f9-4495-af40-aa221f0b3fa5/4179ae51-cf3a-4bce-929c-a59c2a13f09f/f3a16da1-c1d9-43a4-8a05-0965021b6865"
-          (reference "R15") (unit 1)
-        )
-        (path "/3c8df2a5-e9f9-4495-af40-aa221f0b3fa5/4179ae51-cf3a-4bce-929c-a59c2a13f09f/162d0e00-6252-4458-837d-88970c658cfc"
-          (reference "R17") (unit 1)
-        )
-        (path "/3c8df2a5-e9f9-4495-af40-aa221f0b3fa5/8cd80f45-633d-420a-bdbe-39ad6abe5b0e/f3a16da1-c1d9-43a4-8a05-0965021b6865"
-          (reference "R19") (unit 1)
-        )
-        (path "/3c8df2a5-e9f9-4495-af40-aa221f0b3fa5/8cd80f45-633d-420a-bdbe-39ad6abe5b0e/162d0e00-6252-4458-837d-88970c658cfc"
-          (reference "R21") (unit 1)
+          (reference "R18") (unit 1)
+        )
+        (path "/3c8df2a5-e9f9-4495-af40-aa221f0b3fa5/4179ae51-cf3a-4bce-929c-a59c2a13f09f/162d0e00-6252-4458-837d-88970c658cfc"
+          (reference "R20") (unit 1)
+        )
+        (path "/3c8df2a5-e9f9-4495-af40-aa221f0b3fa5/8cd80f45-633d-420a-bdbe-39ad6abe5b0e/f3a16da1-c1d9-43a4-8a05-0965021b6865"
+          (reference "R22") (unit 1)
+        )
+        (path "/3c8df2a5-e9f9-4495-af40-aa221f0b3fa5/8cd80f45-633d-420a-bdbe-39ad6abe5b0e/162d0e00-6252-4458-837d-88970c658cfc"
+          (reference "R24") (unit 1)
         )
       )
@@
   (symbol (lib_id "Device:C") (at 100.33 76.2 180) (unit 1)
     (in_bom yes) (on_board yes) (dnp no)
-    (property "Reference" "C22" (at 95.25 74.93 0)
+    (property "Reference" "C13" (at 95.25 74.93 0)
       (effects (font (size 1.27 1.27)) (justify right))
     )
@@
       (project "crossover"
         (path "/3c8df2a5-e9f9-4495-af40-aa221f0b3fa5/4179ae51-cf3a-4bce-929c-a59c2a13f09f/f3a16da1-c1d9-43a4-8a05-0965021b6865"
-          (reference "C22") (unit 1)
-        )
-        (path "/3c8df2a5-e9f9-4495-af40-aa221f0b3fa5/4179ae51-cf3a-4bce-929c-a59c2a13f09f/162d0e00-6252-4458-837d-88970c658cfc"
-          (reference "C23") (unit 1)
-        )
-        (path "/3c8df2a5-e9f9-4495-af40-aa221f0b3fa5/8cd80f45-633d-420a-bdbe-39ad6abe5b0e/f3a16da1-c1d9-43a4-8a05-0965021b6865"
-          (reference "C24") (unit 1)
-        )
-        (path "/3c8df2a5-e9f9-4495-af40-aa221f0b3fa5/8cd80f45-633d-420a-bdbe-39ad6abe5b0e/162d0e00-6252-4458-837d-88970c658cfc"
-          (reference "C25") (unit 1)
+          (reference "C13") (unit 1)
+        )
+        (path "/3c8df2a5-e9f9-4495-af40-aa221f0b3fa5/4179ae51-cf3a-4bce-929c-a59c2a13f09f/162d0e00-6252-4458-837d-88970c658cfc"
+          (reference "C15") (unit 1)
+        )
+        (path "/3c8df2a5-e9f9-4495-af40-aa221f0b3fa5/8cd80f45-633d-420a-bdbe-39ad6abe5b0e/f3a16da1-c1d9-43a4-8a05-0965021b6865"
+          (reference "C17") (unit 1)
+        )
+        (path "/3c8df2a5-e9f9-4495-af40-aa221f0b3fa5/8cd80f45-633d-420a-bdbe-39ad6abe5b0e/162d0e00-6252-4458-837d-88970c658cfc"
+          (reference "C19") (unit 1)
         )
       )
@@
   (symbol (lib_id "Device:R") (at 95.25 66.04 90) (unit 1)
     (in_bom yes) (on_board yes) (dnp no) (fields_autoplaced)
-    (property "Reference" "R16" (at 95.25 59.69 90)
+    (property "Reference" "R19" (at 95.25 59.69 90)
       (effects (font (size 1.27 1.27)))
     )
@@
       (project "crossover"
         (path "/3c8df2a5-e9f9-4495-af40-aa221f0b3fa5/4179ae51-cf3a-4bce-929c-a59c2a13f09f/f3a16da1-c1d9-43a4-8a05-0965021b6865"
-          (reference "R16") (unit 1)
-        )
-        (path "/3c8df2a5-e9f9-4495-af40-aa221f0b3fa5/4179ae51-cf3a-4bce-929c-a59c2a13f09f/162d0e00-6252-4458-837d-88970c658cfc"
-          (reference "R18") (unit 1)
-        )
-        (path "/3c8df2a5-e9f9-4495-af40-aa221f0b3fa5/8cd80f45-633d-420a-bdbe-39ad6abe5b0e/f3a16da1-c1d9-43a4-8a05-0965021b6865"
-          (reference "R20") (unit 1)
-        )
-        (path "/3c8df2a5-e9f9-4495-af40-aa221f0b3fa5/8cd80f45-633d-420a-bdbe-39ad6abe5b0e/162d0e00-6252-4458-837d-88970c658cfc"
-          (reference "R22") (unit 1)
-        )
-      )
+          (reference "R19") (unit 1)
+        )
+        (path "/3c8df2a5-e9f9-4495-af40-aa221f0b3fa5/4179ae51-cf3a-4bce-929c-a59c2a13f09f/162d0e00-6252-4458-837d-88970c658cfc"
+          (reference "R21") (unit 1)
+        )
+        (path "/3c8df2a5-e9f9-4495-af40-aa221f0b3fa5/8cd80f45-633d-420a-bdbe-39ad6abe5b0e/f3a16da1-c1d9-43a4-8a05-0965021b6865"
+          (reference "R23") (unit 1)
+        )
+        (path "/3c8df2a5-e9f9-4495-af40-aa221f0b3fa5/8cd80f45-633d-420a-bdbe-39ad6abe5b0e/162d0e00-6252-4458-837d-88970c658cfc"
+          (reference "R25") (unit 1)
+        )
+      )

Commit message: Switch to TL074
Parts:
- U2: renamed from U4; value TL072 -> TL074; footprint Package_DIP:DIP-8_W7.62mm_Socket -> (none); symbol Amplifier_Operational:TL072 -> Amplifier_Operational:TL074
Connections:
- net out: now also U2.8, U2.9 (-); no longer U2.1, U2.2 (-)
- net at C13.2, R19.2: now also U2.10 (+); no longer U2.3 (+)
Changed lines of the file:
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@@
     )
   )
-  (symbol (lib_id "Amplifier_Operational:TL072") (at 111.76 68.58 0) (unit 1)
+  (symbol (lib_id "Amplifier_Operational:TL074") (at 111.76 68.58 0) (unit 3)
     (in_bom yes) (on_board yes) (dnp no) (fields_autoplaced)
-    (property "Reference" "U4" (at 111.76 58.42 0)
-      (effects (font (size 1.27 1.27)))
+    (property "Reference" "U2" (at 111.76 63.5 0)
+      (effects (font (size 1.27 1.27)) (justify left))
     )
-    (property "Value" "TL072" (at 111.76 60.96 0)
-      (effects (font (size 1.27 1.27)))
+    (property "Value" "TL074" (at 111.76 73.66 0)
+      (effects (font (size 1.27 1.27)) (justify left))
     )
-    (property "Footprint" "Package_DIP:DIP-8_W7.62mm_Socket" (at 111.76 68.58 0)
+    (property "Footprint" "" (at 110.49 66.04 0)
       (effects (font (size 1.27 1.27)) hide)
     )
-    (property "Datasheet" "http://www.ti.com/lit/ds/symlink/tl071.pdf" (at 111.76 68.58 0)
+    (property "Datasheet" "http://www.ti.com/lit/ds/symlink/tl071.pdf" (at 113.03 63.5 0)
       (effects (font (size 1.27 1.27)) hide)
     )
@@
     (pin "6")
     (pin "7")
+    (pin "10")
+    (pin "8")
+    (pin "9")
+    (pin "12")
+    (pin "13")
+    (pin "14")
+    (pin "11")
     (pin "4")
-    (pin "8")
     (instances
       (project "crossover"
         (path "/3c8df2a5-e9f9-4495-af40-aa221f0b3fa5/4179ae51-cf3a-4bce-929c-a59c2a13f09f/f3a16da1-c1d9-43a4-8a05-0965021b6865"
-          (reference "U4") (unit 1)
+          (reference "U2") (unit 3)
         )
         (path "/3c8df2a5-e9f9-4495-af40-aa221f0b3fa5/4179ae51-cf3a-4bce-929c-a59c2a13f09f/162d0e00-6252-4458-837d-88970c658cfc"
-          (reference "U4") (unit 2)
+          (reference "U2") (unit 4)
         )
         (path "/3c8df2a5-e9f9-4495-af40-aa221f0b3fa5/8cd80f45-633d-420a-bdbe-39ad6abe5b0e/f3a16da1-c1d9-43a4-8a05-0965021b6865"
-          (reference "U5") (unit 1)
+          (reference "U3") (unit 3)
         )
         (path "/3c8df2a5-e9f9-4495-af40-aa221f0b3fa5/8cd80f45-633d-420a-bdbe-39ad6abe5b0e/162d0e00-6252-4458-837d-88970c658cfc"
-          (reference "U5") (unit 2)
+          (reference "U3") (unit 4)
         )
       )

Commit message: Assign footprints to everything
Parts:
- R18, R19: footprint Resistor_THT:R_Axial_DIN0207_L6.3mm_D2.5mm_P7.62mm_Horizontal -> Resistor_SMD:R_1206_3216Metric_Pad1.30x1.75mm_HandSolder
- U2: footprint (none) -> Package_SO:SOIC-14-16_3.9x9.9mm_P1.27mm
Changed lines of the file:
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@@
       (effects (font (size 1.27 1.27)) (justify left))
     )
-    (property "Footprint" "" (at 110.49 66.04 0)
+    (property "Footprint" "Package_SO:SOIC-14-16_3.9x9.9mm_P1.27mm" (at 110.49 66.04 0)
       (effects (font (size 1.27 1.27)) hide)
     )
@@
       (effects (font (size 1.27 1.27)))
     )
-    (property "Footprint" "Resistor_THT:R_Axial_DIN0207_L6.3mm_D2.5mm_P7.62mm_Horizontal" (at 80.01 67.818 90)
+    (property "Footprint" "Resistor_SMD:R_1206_3216Metric_Pad1.30x1.75mm_HandSolder" (at 80.01 67.818 90)
       (effects (font (size 1.27 1.27)) hide)
     )
@@
       (effects (font (size 1.27 1.27)))
     )
-    (property "Footprint" "Resistor_THT:R_Axial_DIN0207_L6.3mm_D2.5mm_P7.62mm_Horizontal" (at 95.25 67.818 90)
+    (property "Footprint" "Resistor_SMD:R_1206_3216Metric_Pad1.30x1.75mm_HandSolder" (at 95.25 67.818 90)
       (effects (font (size 1.27 1.27)) hide)
     )

Commit message: Finish placing
Parts:
- U2: footprint Package_SO:SOIC-14-16_3.9x9.9mm_P1.27mm -> Package_SO:SOIC-14_3.9x8.7mm_P1.27mm
Changed lines of the file:
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@@
       (effects (font (size 1.27 1.27)) (justify left))
     )
-    (property "Footprint" "Package_SO:SOIC-14-16_3.9x9.9mm_P1.27mm" (at 110.49 66.04 0)
+    (property "Footprint" "Package_SO:SOIC-14_3.9x8.7mm_P1.27mm" (at 110.49 66.04 0)
       (effects (font (size 1.27 1.27)) hide)
     )
