File: buffer.kicad_sch (KiCad schematic)
At the start: 3 parts, among them U1 TL072

Commit message: Fix input section
Parts:
- removed R3: 1K, Resistor_THT:R_Axial_DIN0207_L6.3mm_D2.5mm_P7.62mm_Horizontal, symbol Device:R
- removed R4: 100K, Resistor_THT:R_Axial_DIN0207_L6.3mm_D2.5mm_P7.62mm_Horizontal, symbol Device:R
- added C33: 4.7uF, symbol Device:C_Polarized_US
- added C35: 1n, symbol Device:C
- added R36, R38: 22K, symbol Device:R
- added R40: 100, symbol Device:R
Connections:
- net GNDREF: now also R38.2
- net In: now also R40.1
- net at U1.3 (+): now also C33.2, R38.1
- new net: C33.1, C35.1, R36.1, R40.2
- new net VDD: C35.2, R36.2
Other:
- moved on the sheet: U1A

Commit message: Re-annotate and run erc
Parts:
- renumbered C35 to C1, C33 to C2, R40 to R4, R36 to R5, R38 to R6
Changed lines of the file:
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@@
   (symbol (lib_id "Device:R") (at 88.9 57.15 0) (unit 1)
     (in_bom yes) (on_board yes) (dnp no) (fields_autoplaced)
-    (property "Reference" "R38" (at 91.44 56.515 0)
+    (property "Reference" "R6" (at 91.44 56.515 0)
       (effects (font (size 1.27 1.27)) (justify left))
     )
@@
       (project "crossover"
         (path "/3c8df2a5-e9f9-4495-af40-aa221f0b3fa5/87eeb169-ec39-4325-b98a-d89c839087c5"
-          (reference "R38") (unit 1)
+          (reference "R6") (unit 1)
         )
         (path "/3c8df2a5-e9f9-4495-af40-aa221f0b3fa5/cd09c5f7-2b82-443b-9511-5215bae1a227"
-          (reference "R39") (unit 1)
+          (reference "R9") (unit 1)
         )
       )
@@
   (symbol (lib_id "Device:R") (at 43.18 58.42 0) (unit 1)
     (in_bom yes) (on_board yes) (dnp no) (fields_autoplaced)
-    (property "Reference" "R36" (at 45.72 57.785 0)
+    (property "Reference" "R5" (at 45.72 57.785 0)
       (effects (font (size 1.27 1.27)) (justify left))
     )
@@
       (project "crossover"
         (path "/3c8df2a5-e9f9-4495-af40-aa221f0b3fa5/87eeb169-ec39-4325-b98a-d89c839087c5"
-          (reference "R36") (unit 1)
+          (reference "R5") (unit 1)
         )
         (path "/3c8df2a5-e9f9-4495-af40-aa221f0b3fa5/cd09c5f7-2b82-443b-9511-5215bae1a227"
-          (reference "R37") (unit 1)
+          (reference "R8") (unit 1)
         )
       )
@@
   (symbol (lib_id "power:VDD") (at 43.18 69.85 180) (unit 1)
     (in_bom yes) (on_board yes) (dnp no) (fields_autoplaced)
-    (property "Reference" "#PWR031" (at 43.18 66.04 0)
+    (property "Reference" "#PWR05" (at 43.18 66.04 0)
       (effects (font (size 1.27 1.27)) hide)
     )
@@
       (project "crossover"
         (path "/3c8df2a5-e9f9-4495-af40-aa221f0b3fa5/87eeb169-ec39-4325-b98a-d89c839087c5"
-          (reference "#PWR031") (unit 1)
+          (reference "#PWR05") (unit 1)
         )
         (path "/3c8df2a5-e9f9-4495-af40-aa221f0b3fa5/cd09c5f7-2b82-443b-9511-5215bae1a227"
-          (reference "#PWR032") (unit 1)
+          (reference "#PWR07") (unit 1)
         )
       )
@@
   (symbol (lib_id "Device:C_Polarized_US") (at 68.58 46.99 90) (unit 1)
     (in_bom yes) (on_board yes) (dnp no) (fields_autoplaced)
-    (property "Reference" "C33" (at 67.945 40.64 90)
+    (property "Reference" "C2" (at 67.945 40.64 90)
       (effects (font (size 1.27 1.27)))
     )
@@
       (project "crossover"
         (path "/3c8df2a5-e9f9-4495-af40-aa221f0b3fa5/87eeb169-ec39-4325-b98a-d89c839087c5"
-          (reference "C33") (unit 1)
+          (reference "C2") (unit 1)
         )
         (path "/3c8df2a5-e9f9-4495-af40-aa221f0b3fa5/cd09c5f7-2b82-443b-9511-5215bae1a227"
-          (reference "C34") (unit 1)
+          (reference "C4") (unit 1)
         )
       )
@@
   (symbol (lib_id "Device:C") (at 54.61 58.42 0) (unit 1)
     (in_bom yes) (on_board yes) (dnp no) (fields_autoplaced)
-    (property "Reference" "C35" (at 58.42 57.785 0)
+    (property "Reference" "C1" (at 58.42 57.785 0)
       (effects (font (size 1.27 1.27)) (justify left))
     )
@@
       (project "crossover"
         (path "/3c8df2a5-e9f9-4495-af40-aa221f0b3fa5/87eeb169-ec39-4325-b98a-d89c839087c5"
-          (reference "C35") (unit 1)
+          (reference "C1") (unit 1)
         )
         (path "/3c8df2a5-e9f9-4495-af40-aa221f0b3fa5/cd09c5f7-2b82-443b-9511-5215bae1a227"
-          (reference "C36") (unit 1)
+          (reference "C3") (unit 1)
         )
       )
@@
   (symbol (lib_id "Device:R") (at 35.56 46.99 90) (unit 1)
     (in_bom yes) (on_board yes) (dnp no) (fields_autoplaced)
-    (property "Reference" "R40" (at 35.56 41.91 90)
+    (property "Reference" "R4" (at 35.56 41.91 90)
       (effects (font (size 1.27 1.27)))
     )
@@
       (project "crossover"
         (path "/3c8df2a5-e9f9-4495-af40-aa221f0b3fa5/87eeb169-ec39-4325-b98a-d89c839087c5"
-          (reference "R40") (unit 1)
+          (reference "R4") (unit 1)
         )
         (path "/3c8df2a5-e9f9-4495-af40-aa221f0b3fa5/cd09c5f7-2b82-443b-9511-5215bae1a227"
-          (reference "R41") (unit 1)
+          (reference "R7") (unit 1)
         )
       )
@@
   (symbol (lib_id "power:GNDREF") (at 88.9 67.31 0) (unit 1)
     (in_bom yes) (on_board yes) (dnp no) (fields_autoplaced)
-    (property "Reference" "#PWR033" (at 88.9 73.66 0)
+    (property "Reference" "#PWR06" (at 88.9 73.66 0)
       (effects (font (size 1.27 1.27)) hide)
     )
@@
       (project "crossover"
         (path "/3c8df2a5-e9f9-4495-af40-aa221f0b3fa5/87eeb169-ec39-4325-b98a-d89c839087c5"
-          (reference "#PWR033") (unit 1)
+          (reference "#PWR06") (unit 1)
         )
         (path "/3c8df2a5-e9f9-4495-af40-aa221f0b3fa5/cd09c5f7-2b82-443b-9511-5215bae1a227"
-          (reference "#PWR034") (unit 1)
+          (reference "#PWR08") (unit 1)
         )
       )

Commit message: Assign footprints to everything
Parts:
- C1: footprint (none) -> Capacitor_SMD:C_0805_2012Metric_Pad1.18x1.45mm_HandSolder
- C2: footprint (none) -> Capacitor_THT:CP_Radial_D5.0mm_P2.00mm
- R4: footprint (none) -> Resistor_THT:R_Axial_DIN0207_L6.3mm_D2.5mm_P7.62mm_Horizontal
- R5, R6: footprint (none) -> Resistor_SMD:R_1206_3216Metric_Pad1.30x1.75mm_HandSolder
Changed lines of the file:
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@@
       (effects (font (size 1.27 1.27)) (justify left))
     )
-    (property "Footprint" "" (at 87.122 57.15 90)
+    (property "Footprint" "Resistor_SMD:R_1206_3216Metric_Pad1.30x1.75mm_HandSolder" (at 87.122 57.15 90)
       (effects (font (size 1.27 1.27)) hide)
     )
@@
       (effects (font (size 1.27 1.27)) (justify left))
     )
-    (property "Footprint" "" (at 41.402 58.42 90)
+    (property "Footprint" "Resistor_SMD:R_1206_3216Metric_Pad1.30x1.75mm_HandSolder" (at 41.402 58.42 90)
       (effects (font (size 1.27 1.27)) hide)
     )
@@
       (effects (font (size 1.27 1.27)))
     )
-    (property "Footprint" "" (at 68.58 46.99 0)
+    (property "Footprint" "Capacitor_THT:CP_Radial_D5.0mm_P2.00mm" (at 68.58 46.99 0)
       (effects (font (size 1.27 1.27)) hide)
     )
@@
       (effects (font (size 1.27 1.27)) (justify left))
     )
-    (property "Footprint" "" (at 55.5752 62.23 0)
+    (property "Footprint" "Capacitor_SMD:C_0805_2012Metric_Pad1.18x1.45mm_HandSolder" (at 55.5752 62.23 0)
       (effects (font (size 1.27 1.27)) hide)
     )
@@
       (effects (font (size 1.27 1.27)))
     )
-    (property "Footprint" "" (at 35.56 48.768 90)
+    (property "Footprint" "Resistor_THT:R_Axial_DIN0207_L6.3mm_D2.5mm_P7.62mm_Horizontal" (at 35.56 48.768 90)
       (effects (font (size 1.27 1.27)) hide)
     )
